File: ZX_Spectrum_Keyboard_Standard/ZX_Spectrum_Keyboard_Standard/ZX_Spectrum_Keyboard_Standard.kicad_pcb (KiCad board)
At the start: 2 copper layers, 210 x 90 mm, 46 parts, among them J1 KB2, J2 KB1

Commit message: Corrected ENTER key location (duh)
Parts:
- moved KB13 171.5 mm to (237.7, 107.8)
- moved KC4 19.0 mm to (85.2, 107.8)
- moved KC5 19.0 mm to (104.3, 107.8)
- moved KC3 19.0 mm to (66.2, 107.8)
- moved KC6 19.0 mm to (123.3, 107.8)
- moved KC10 19.0 mm to (199.5, 107.8)
- moved KC7 19.0 mm to (142.4, 107.8)
- moved KC8 19.0 mm to (161.4, 107.8)
- moved KC9 19.0 mm to (180.5, 107.8)
- moved KC11 19.0 mm to (218.6, 107.8)
- moved KE6 0.09 mm to (232.9, 126.9)
Routing:
- net KBD2: track 244.4 -> 148.9 mm
- net KBD11: track 295.5 -> 255.1 mm
- net KBD12: track 335.8 -> 295.5 mm
- net KBD10: track 262.5 -> 224.6 mm
- net KBD13: track 375.6 -> 353.4 mm
- net KBD5: track 113.7 -> 104.2 mm
- net KBD9: track 194.8 -> 202.6 mm
- net KBD3: track 264.2 -> 258.1 mm
- net KBD7: track 187.8 -> 182.3 mm
- net KBD4: track 128.2 -> 130.4 mm
- net KBD6: track 202.2 -> 200.0 mm
Other:
- board text added: "Rev. B"
