File: ZX80_Gaming_Keyboard/ZX80_Gaming_Keyboard.kicad_pcb (KiCad board)
At the start: 2 copper layers, 276 x 89 mm, 54 parts, among them J1 KB1, J2 KB2, J3 SPACE_ZERO, J4 ZX_ACE, SW1 1, SW10 0, SW11 Q, SW12 W, SW13 E, SW14 R, SW15 T, SW16 Y, SW17 U, SW18 I, SW19 O, SW2 2, SW20 P, SW21 A, SW22 S, SW23 D, SW24 F, SW25 G, SW26 H, SW27 J, SW28 K, SW29 L, SW3 3, SW30 NL, SW31 SHIFT, SW32 Z, SW33 X, SW34 C, SW35 V, SW36 B, SW37 N, SW38 M, SW39 DOT, SW4 4, SW40 SPACE, SW41 LEFT, SW42 DOWN, SW43 UP, SW44 RIGHT, SW45 RUBOUT, SW5 5, SW6 6, SW7 7, SW8 8, SW9 9

Commit message: Rev. C
Removed dedicated DEL key - still need to figure it out
Parts:
- removed D1: 1N4148, Diode_THT:D_DO-35_SOD27_P7.62mm_Horizontal
- removed SW45: RUBOUT, Button_Switch_Keyboard:SW_Cherry_MX_1.00u_PCB
Routing:
- net COL1: track 357.5 -> 0.00 mm, vias 1 -> 0
- net COL3: track 354.4 -> 0.00 mm
- net COL5: track 346.1 -> 0.00 mm, vias 1 -> 0
- net COL2: track 327.4 -> 0.00 mm, vias 1 -> 0
- net COL4: track 287.6 -> 0.00 mm, vias 2 -> 0
- net A11: track 270.0 -> 0.00 mm, vias 2 -> 0
- net A12: track 264.4 -> 0.00 mm, vias 1 -> 0
- net A8: track 255.1 -> 0.00 mm, vias 1 -> 0
- net A15: track 223.6 -> 0.00 mm, vias 1 -> 0
- net A9: track 190.9 -> 0.00 mm, vias 1 -> 0
- net A10: track 173.1 -> 0.00 mm, vias 1 -> 0
- net A14: track 147.8 -> 0.00 mm
- net Net-(J3-Pin_2): track 143.2 -> 0.00 mm, vias 1 -> 0
- net A13: track 112.2 -> 0.00 mm
- net CUR_DOWN: track 73.6 -> 0.00 mm
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