File: ZX80_Gaming_Keyboard/ZX80_Gaming_Keyboard.kicad_pcb (KiCad board)
At the start: 2 copper layers, 276 x 89 mm, 52 parts, among them J1 KB1, J2 KB2, J3 SPACE_ZERO, J4 ZX_ACE, SW1 1, SW10 0, SW11 Q, SW12 W, SW13 E, SW14 R, SW15 T, SW16 Y, SW17 U, SW18 I, SW19 O, SW2 2, SW20 P, SW21 A, SW22 S, SW23 D, SW24 F, SW25 G, SW26 H, SW27 J, SW28 K, SW29 L, SW3 3, SW30 NL, SW31 SHIFT, SW32 Z, SW33 X, SW34 C, SW35 V, SW36 B, SW37 N, SW38 M, SW39 DOT, SW4 4, SW40 SPACE, SW41 LEFT, SW42 DOWN, SW43 UP, SW44 RIGHT, SW5 5, SW6 6, SW7 7, SW8 8, SW9 9

Commit message: Corrected keyswitch placement
Key switches were too close together, duh
Parts:
- added J5: ZX80 Joypad, Connector_PinHeader_2.54mm:PinHeader_1x07_P2.54mm_Vertical, F.Cu at (333.2, 147.1)
- SW1, SW10, SW11, SW12, SW13, SW14, SW15, SW16, SW17, SW18, SW19, SW2, SW20, SW21, SW22, SW23, SW24, SW25, SW26, SW27, SW28, SW29, SW3, SW30, SW31, SW32, SW33, SW34, SW35, SW36, SW37, SW38, SW39, SW4, SW40, SW41, SW42, SW43, SW44, SW5, SW6, SW7, SW8, SW9: footprint Button_Switch_Keyboard:SW_Cherry_MX_1.00u_PCB -> Button_Switch_THT:SW_PUSH-12mm
- moved SW30 53.9 mm to (234.7, 152.1)
- moved SW29 50.8 mm to (218.7, 152.1)
- moved SW20 49.5 mm to (234.7, 136.1)
- moved SW44 49.0 mm to (282.7, 168.1)
- moved SW28 47.8 mm to (202.7, 152.1)
- moved SW19 46.5 mm to (218.7, 136.1)
- moved SW42 46.0 mm to (266.7, 168.1)
- moved SW43 45.8 mm to (266.7, 152.1)
- moved SW27 44.7 mm to (186.7, 152.1)
- moved SW18 43.4 mm to (202.7, 136.1)
- moved SW41 43.0 mm to (250.7, 168.1)
- moved J4 41.8 mm to (293.4, 117.6)
- moved J3 41.8 mm to (303.6, 117.6)
- moved SW26 41.7 mm to (170.7, 152.1)
- moved SW17 40.4 mm to (186.7, 136.1)
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Connections:
- net A10 renamed /A10
- net A11 renamed /A11
- net A12 renamed /A12
- net A13 renamed /A13
- net A14 renamed /A14
- net A15 renamed /A15
- net A8 renamed /A8
- net A9 renamed /A9
- net COL3 renamed /COL3
- net CUR_DOWN renamed /CUR_DOWN
- net CUR_UP renamed /CUR_UP
- J1 pad 1: COL1 -> /COL1
- J1 pad 2: COL2 -> /COL2
- J1 pad 4: COL4 -> /COL4
- J1 pad 5: COL5 -> /COL5
- J4 pad 1: COL1 -> /COL1
- J4 pad 4: COL2 -> /COL2
- SW1 pad 1: COL5 -> /COL1
- SW10 pad 1: COL5 -> /COL1
- SW11 pad 1: COL5 -> /COL1
- SW12 pad 1: COL4 -> /COL2
- SW14 pad 1: COL2 -> /COL4
- SW15 pad 1: COL1 -> /COL5
- SW16 pad 1: COL1 -> /COL5
- SW17 pad 1: COL2 -> /COL4
- SW19 pad 1: COL4 -> /COL2
- SW2 pad 1: COL4 -> /COL2
- SW20 pad 1: COL5 -> /COL1
- SW21 pad 1: COL5 -> /COL1
- SW22 pad 1: COL4 -> /COL2
- SW24 pad 1: COL2 -> /COL4
- SW25 pad 1: COL1 -> /COL5
- SW26 pad 1: COL1 -> /COL5
- SW27 pad 1: COL2 -> /COL4
- SW29 pad 1: COL4 -> /COL2
- SW30 pad 1: COL5 -> /COL1
- SW31 pad 1: COL5 -> /COL1
- SW32 pad 1: COL4 -> /COL2
- SW34 pad 1: COL2 -> /COL4
- SW35 pad 1: COL1 -> /COL5
- SW36 pad 1: COL1 -> /COL5
- SW37 pad 1: COL2 -> /COL4
- SW39 pad 1: COL4 -> /COL2
- SW4 pad 1: COL2 -> /COL4
- SW40 pad 1: COL5 -> /COL1
- SW41 pad 1: COL1 -> /COL1
- SW5 pad 1: COL1 -> /COL5
- SW6 pad 1: COL1 -> /COL5
- SW7 pad 1: COL2 -> /COL4
- SW9 pad 1: COL4 -> /COL2
Other:
- board text added: "Rev. D"
- board text removed: "Rev. C"
