File: ZX80_Gaming_Keyboard/ZX80_Gaming_Keyboard.kicad_sch (KiCad schematic)
At the start: 54 parts, among them J1 KB1, J2 KB2, J3 SPACE_ZERO, J4 ZX_ACE, SW1 1, SW10 0, SW11 Q, SW12 W, SW13 E, SW14 R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

Commit message: Rev. C
Removed dedicated DEL key - still need to figure it out
Parts:
- removed D1: 1N4148, Diode_THT:D_DO-35_SOD27_P7.62mm_Horizontal, symbol Device:D
- removed SW45: RUBOUT, Button_Switch_Keyboard:SW_Cherry_MX_1.00u_PCB, symbol Switch:SW_Push_45deg
