File: ZX80_Gaming_Keyboard/ZX80_Gaming_Keyboard.kicad_sch (KiCad schematic)
At the start: 52 parts, among them J1 KB1, J2 KB2, J3 SPACE_ZERO, J4 ZX_ACE, SW1 1, SW10 0, SW11 Q, SW12 W, SW13 E, SW14 R, SW15 T, SW16 Y, SW17 U, SW18 I, SW19 O, SW2 2, SW20 P, SW21 A, SW22 S, SW23 D, SW24 F, SW25 G, SW26 H, SW27 J, SW28 K, SW29 L, SW3 3, SW30 NL, SW31 SHIFT, SW32 Z, SW33 X, SW34 C, SW35 V, SW36 B, SW37 N, SW38 M, SW39 DOT, SW4 4, SW40 SPACE, SW41 LEFT, SW42 DOWN, SW43 UP, SW44 RIGHT, SW5 5, SW6 6, SW7 7, SW8 8, SW9 9

Commit message: Corrected keyswitch placement
Key switches were too close together, duh
Parts:
- added J5: ZX80 Joypad, Connector_PinHeader_2.54mm:PinHeader_1x07_P2.54mm_Vertical, symbol Connector_Generic:Conn_01x07
- SW1, SW10, SW11, SW12, SW13, SW14, SW15, SW16, SW17, SW18, SW19, SW2, SW20, SW21, SW22, SW23, SW24, SW25, SW26, SW27, SW28, SW29, SW3, SW30, SW31, SW32, SW33, SW34, SW35, SW36, SW37, SW38, SW39, SW4, SW40, SW41, SW42, SW43, SW44, SW5, SW6, SW7, SW8, SW9: footprint Button_Switch_Keyboard:SW_Cherry_MX_1.00u_PCB -> Button_Switch_THT:SW_PUSH-12mm
Connections:
- net A11: now also J5.3 (Pin_3)
- net A12: now also J5.5 (Pin_5)
- net A15: now also J5.7 (Pin_7)
- net COL1: now also SW1.1, SW10.1, SW11.1, SW20.1, SW21.1, SW30.1, SW31.1, SW40.1, J5.1 (Pin_1); no longer SW15.1, SW16.1, SW25.1, SW26.1, SW35.1, SW36.1, SW5.1, SW6.1
- net COL2: now also SW12.1, SW19.1, SW2.1, SW22.1, SW29.1, SW32.1, SW39.1, SW9.1, J5.2 (Pin_2); no longer SW14.1, SW17.1, SW24.1, SW27.1, SW34.1, SW37.1, SW4.1, SW7.1
- net COL3: now also J5.4 (Pin_4)
- net COL4: now also SW14.1, SW17.1, SW24.1, SW27.1, SW34.1, SW37.1, SW4.1, SW7.1; no longer SW12.1, SW19.1, SW2.1, SW22.1, SW29.1, SW32.1, SW39.1, SW9.1
- net COL5: now also SW15.1, SW16.1, SW25.1, SW26.1, SW35.1, SW36.1, SW5.1, SW6.1, J5.6 (Pin_6); no longer SW1.1, SW10.1, SW11.1, SW20.1, SW21.1, SW30.1, SW31.1, SW40.1
