File: ZX_Spectrum_Next_Keyboard/Spectrum_Next_Keyboard/Spectrum_Next_Keyboard.kicad_pcb (KiCad board)
At the start: 2 copper layers, 61 parts, among them J1 TOP, J2 BOT, J3 2PIN

Commit message: Initial design completed
Parts:
- added H1: MountingHole, MountingHole:MountingHole_3.2mm_M3, F.Cu at (21.6, 47.0)
- added H2: MountingHole, MountingHole:MountingHole_3.2mm_M3, F.Cu at (149.7, 47.0)
- added H3: MountingHole, MountingHole:MountingHole_3.2mm_M3, F.Cu at (21.6, 150.1)
- added H4: MountingHole, MountingHole:MountingHole_3.2mm_M3, F.Cu at (277.6, 47.0)
- added H5: MountingHole, MountingHole:MountingHole_3.2mm_M3, F.Cu at (149.7, 150.1)
- added H6: MountingHole, MountingHole:MountingHole_3.2mm_M3, F.Cu at (277.6, 150.1)
- moved J1 138.9 mm to (175.5, 46.9), turned to -90 degrees
- moved J2 32.9 mm to (90.4, 46.9)
- moved J3 18.7 mm to (253.0, 46.9), turned to -90 degrees
- moved KB13 2.50 mm to (260.7, 99.3)
- moved KB11 2.50 mm to (231.9, 79.9)
- moved KB12 2.50 mm to (251.0, 79.9)
- moved KB4 2.50 mm to (98.6, 79.9)
- moved KB5 2.50 mm to (117.6, 79.9)
- moved KB6 2.50 mm to (136.7, 79.9)
- moved KB7 2.50 mm to (155.7, 79.9)
- moved KB8 2.50 mm to (174.8, 79.9)
- moved KB9 2.50 mm to (193.8, 79.9)
- moved KE3 2.50 mm to (70.0, 137.1)
- moved KE4 2.50 mm to (89.1, 137.1)
- moved KE6 2.50 mm to (158.1, 137.1)
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Connections:
- net COL1 renamed /COL1
- net COL2 renamed /COL2
- net COL3 renamed /COL3
- net COL4 renamed /COL4
- net COL5 renamed /COL5
- net COL6 renamed /COL6
- net COL7 renamed /COL7
- net COL8 renamed /COL8
- net ROW1 renamed /ROW1
- net ROW2 renamed /ROW2
- net ROW3 renamed /ROW3
- net ROW4 renamed /ROW4
- net ROW5 renamed /ROW5
- net ROW6 renamed /ROW6
- net ROW7 renamed /ROW7
Routing:
- net /COL4: track 224.9 -> 447.4 mm, vias 0 -> 1
- net /COL8: track 271.7 -> 478.5 mm
- net /COL6: track 225.4 -> 411.5 mm
- net /ROW7: track 296.8 -> 460.4 mm
- net /ROW6: track 302.0 -> 450.4 mm
- net /COL5: track 196.7 -> 323.9 mm
- net /COL7: track 167.8 -> 235.7 mm
- net /ROW2: track 375.0 -> 423.4 mm
- net /ROW1: track 447.1 -> 414.8 mm
- net /ROW5: track 171.1 -> 195.9 mm
- net /COL1: track 150.1 -> 165.5 mm
- net /COL2: track 169.9 -> 183.4 mm
- net /COL3: track 191.7 -> 202.7 mm
- net /ROW3: track 247.8 -> 257.7 mm
- net /ROW4: track 217.6 -> 224.9 mm
Other:
- board outline added: 263.5 x 111 mm
- board text added: "1 2 3 4 5"
- board text added: "7 6"
- board text added: "8 7 6 5 4 3 2 1"
- board text added: "Brett Hallen, Jan 2026"
- board text added: "Columns"
- board text added: "Rows"
- board text added: "ZX Spectrum Next"

Commit message: Added NumPad to keyboard
Parts:
- added H7: MountingHole, MountingHole:MountingHole_3.2mm_M3, F.Cu at (383.1, 71.1)
- added H8: MountingHole, MountingHole:MountingHole_3.2mm_M3, F.Cu at (383.1, 174.1)
- added KC12: ENTER, Clueless_Engineer:SW_Gateron_LowProfile_THT, F.Cu at (302.4, 103.9)
- added KE10: SPACE, Clueless_Engineer:SW_Gateron_LowProfile_THT, F.Cu at (212.0, 161.1)
- added NP1: 1, Clueless_Engineer:SW_Gateron_LowProfile_THT, F.Cu at (331.0, 142.0)
- added NP10: 0, Clueless_Engineer:SW_Gateron_LowProfile_THT, F.Cu at (331.0, 161.1)
- added NP11: ., Clueless_Engineer:SW_Gateron_LowProfile_THT, F.Cu at (350.1, 161.1)
- added NP12: ENTER, Clueless_Engineer:SW_Gateron_LowProfile_THT, F.Cu at (369.1, 161.1)
- added NP2: 2, Clueless_Engineer:SW_Gateron_LowProfile_THT, F.Cu at (350.1, 142.0)
- added NP3: 3, Clueless_Engineer:SW_Gateron_LowProfile_THT, F.Cu at (369.1, 142.0)
- added NP4: 4, Clueless_Engineer:SW_Gateron_LowProfile_THT, F.Cu at (331.0, 123.0)
- added NP5: 5, Clueless_Engineer:SW_Gateron_LowProfile_THT, F.Cu at (350.1, 123.0)
- added NP6: 6, Clueless_Engineer:SW_Gateron_LowProfile_THT, F.Cu at (369.1, 123.0)
- added NP7: 7, Clueless_Engineer:SW_Gateron_LowProfile_THT, F.Cu at (331.0, 103.9)
- added NP8: 8, Clueless_Engineer:SW_Gateron_LowProfile_THT, F.Cu at (350.1, 103.9)
- added NP9: 9, Clueless_Engineer:SW_Gateron_LowProfile_THT, F.Cu at (369.1, 103.9)
- moved KE13 42.3 mm to (300.1, 161.1)
- moved KD11 42.3 mm to (290.5, 142.0)
- moved KA13 42.3 mm to (297.7, 84.9)
- moved KB13 42.0 mm to (295.3, 123.0)
- moved KE9 40.3 mm to (278.6, 161.1)
- moved KE8 40.3 mm to (259.6, 161.1)
- moved KC1 40.3 mm to (69.1, 123.0)
- moved KD10 40.3 mm to (259.6, 142.0)
- moved KC11 40.3 mm to (269.1, 123.0)
- moved KD4 40.3 mm to (145.3, 142.0)
- moved KA1 40.3 mm to (64.3, 84.9)
- moved KA11 40.3 mm to (254.8, 84.9)
- moved KA4 40.3 mm to (121.5, 84.9)
- moved KA6 40.3 mm to (159.6, 84.9)
- moved KA7 40.3 mm to (178.6, 84.9)
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Routing:
- net /ROW5: track 195.9 -> 650.8 mm, vias 0 -> 1
- net /ROW2: track 423.4 -> 628.9 mm
- net /ROW3: track 257.7 -> 444.7 mm, vias 0 -> 1
- net /COL4: track 447.4 -> 588.2 mm
- net /ROW4: track 224.9 -> 354.3 mm, vias 0 -> 1
- net /ROW1: track 414.8 -> 535.0 mm, vias 1 -> 0
- net /COL7: track 235.7 -> 334.2 mm, vias 0 -> 1
- net /COL5: track 323.9 -> 414.6 mm
- net Net-(NP1-Pad2): track 0.00 -> 80.3 mm
- net /ROW7: track 460.4 -> 533.1 mm
- net /COL8: track 478.5 -> 510.1 mm, vias 0 -> 2
- net /COL6: track 411.5 -> 419.3 mm, vias 0 -> 1
- net /ROW6: track 450.4 -> 455.2 mm
Other:
- board size 263.5 x 111 mm -> 336.5 x 112 mm
- board text added: "Next"
- board text added: "ZX Spectrum"
- board text removed: "ZX Spectrum Next"

Commit message: Rerouted so no vias required
Parts:
- moved J1 17.9 mm to (190.0, 71.0), turned to 90 degrees
- moved J3 2.75 mm to (282.7, 71.1), turned to 90 degrees
Routing:
- net /ROW5: track 650.8 -> 448.4 mm, vias 1 -> 0
- net /ROW1: track 535.0 -> 674.2 mm
- net /ROW2: track 628.9 -> 499.5 mm
- net /COL8: track 510.1 -> 386.6 mm, vias 2 -> 0
- net /COL6: track 419.3 -> 316.4 mm, vias 1 -> 0
- net /ROW6: track 455.2 -> 520.0 mm
- net /COL5: track 414.6 -> 455.9 mm
- net /COL4: track 588.2 -> 563.6 mm, vias 1 -> 0
- net /ROW3: track 444.7 -> 421.3 mm, vias 1 -> 0
- net /COL1: track 165.5 -> 144.8 mm
- net /COL2: track 183.4 -> 167.1 mm
- net /ROW4: track 354.3 -> 367.7 mm, vias 1 -> 0
- net /COL3: track 202.7 -> 189.7 mm
- net /COL7: track 334.2 -> 341.3 mm, vias 1 -> 0
- net /ROW7: track 533.1 -> 530.8 mm
Other:
- board text added: "1 2 3 4 5 6 7 8"
- board text added: "6 7"
- board text removed: "7 6"
- board text removed: "8 7 6 5 4 3 2 1"
