File: ZX80_Joypad/ZX80_Joypad.kicad_pcb (KiCad board)
At the start: 2 copper layers, 100 x 50 mm, 12 parts, among them J1 Conn_02x04_Odd_Even, J2 ZX/ACE Switch, SW1 5/LEFT, SW2 7/UP, SW3 6/DOWN, SW4 8/RIGHT, SW5 ZERO, SW6 SPACE

Commit message: Switched to DE9 connector
Parts:
- removed J1: Conn_02x04_Odd_Even, Connector_PinHeader_2.54mm:PinHeader_2x04_P2.54mm_Vertical
- added J3: DE9_Socket, Connector_Dsub:DSUB-9_Socket_EdgeMount_P2.77mm, F.Cu at (137.3, 82.2)
Routing:
- net /COL1: track 89.3 -> 150.1 mm
- net /UP: track 75.0 -> 104.7 mm
- net /DOWN: track 95.5 -> 76.0 mm
- net /COL3: track 47.0 -> 33.3 mm
- net /COL2: track 18.2 -> 31.8 mm
- net /A11: track 64.3 -> 51.2 mm
- net /COL5: track 49.3 -> 58.9 mm
- net /A12: track 157.6 -> 147.9 mm
- net /A15: track 42.0 -> 49.5 mm
Other:
- board text added: "A12 A15 COL5"
- board text added: "Brett Hallen, Jul 2026"
- board text added: "COL1 A11 COL3 COL2"
- board text removed: "A11 A12 A15"
- board text removed: "Brett Hallen, Jun 2026"
- board text removed: "COL1 COL2 COL3 COL5"
