File: ZX80_Joypad/ZX80_Joypad.kicad_sch (KiCad schematic)
At the start: 12 parts, among them J1 Conn_02x04_Odd_Even, J2 ZX/ACE Switch, SW1 5/LEFT, SW2 7/UP, SW3 6/DOWN, SW4 8/RIGHT, SW5 ZERO, SW6 SPACE

Commit message: Switched to DE9 connector
Parts:
- removed J1: Conn_02x04_Odd_Even, Connector_PinHeader_2.54mm:PinHeader_2x04_P2.54mm_Vertical, symbol Connector_Generic:Conn_02x04_Odd_Even
- added J3: DE9_Socket, Connector_Dsub:DSUB-9_Socket_EdgeMount_P2.77mm, symbol Connector:DE9_Socket
Connections:
- net A11: now also J3.2
- net A12: now also J3.6
- net A15: now also J3.7
- net COL1: now also J3.1
- net COL2: now also J3.5
- net COL3: now also J3.3
- net COL5: now also J3.9
- no-connect marks 1 -> 2
