File: ZX81_Expansion_Breakout/ZX81_Expansion_Breakout.kicad_pcb (KiCad board)
At the start: 2 copper layers, 61.2 x 53.3 mm, 8 parts, among them J1 ZX81 Expansion, J2 Pin Header Breakout, J3 ZX81 Extender, J4 GND LINK, J5 GND LINK, SW1 RESET

Commit message: Tested design
Removed 470Ω current limiting resistor on ~RESET line
Parts:
- removed R1: 470Ω, Resistor_THT:R_Axial_DIN0207_L6.3mm_D2.5mm_P7.62mm_Horizontal
Connections:
- R2 pad 1: Net-(R1-Pad2) -> ~{RESET}
Routing:
- net Net-(R1-Pad2): track 4.85 -> 0.00 mm
- net ~{RESET}: track 47.0 -> 50.5 mm
Other:
- board text added: "Brett Hallen, Oct 2026"
- board text removed: "Brett Hallen, Jul 2026"
Changed lines of the file:
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@@
 	(title_block
 		(title "ZX81 Expansion Breakout")
-		(date "25/JUL/2026")
-		(rev "Issue 1")
+		(date "20/Oct/2026")
+		(rev "Issue 2")
 		(company "Brett Hallen")
 		(comment 3 "https://github.com/zxinfo-diy-electronics/zx81-bus-extender")
@@
 		(embedded_fonts no)
 	)
-	(footprint "Resistor_THT:R_Axial_DIN0207_L6.3mm_D2.5mm_P7.62mm_Horizontal"
-		(layer "F.Cu")
-		(at 111.894 54.857 -90)
-		(descr "Resistor, Axial_DIN0207 series, Axial, Horizontal, pin pitch=7.62mm, 0.25W = 1/4W, length*diameter=6.3*2.5mm^2, http://cdn-reichelt.de/documents/datenblatt/B400/1_4W%23YAG.pdf")
-		(tags "Resistor Axial_DIN0207 series Axial Horizontal pin pitch 7.62mm 0.25W = 1/4W length 6.3mm diameter 2.5mm")
-		(property "Reference" "R1"
-			(at 3.81 -2.37 90)
-			(layer "F.SilkS")
-			(hide yes)
-			(effects
-				(font
-					(size 1 1)
-					(thickness 0.15)
-				)
-			)
-		)
-		(property "Value" "470Ω"
-			(at 3.81 0 90)
-			(layer "F.SilkS")
-			(effects
-				(font
-					(size 1 1)
-				)
-			)
-		)
-		(property "Datasheet" ""
-			(at 0 0 90)
-			(layer "F.Fab")
-			(hide yes)
-			(effects
-				(font
-					(size 1.27 1.27)
-				)
-			)
-		)
-		(property "Description" "Resistor"
-			(at 0 0 90)
-			(layer "F.Fab")
-			(hide yes)
-			(effects
-				(font
-					(size 1.27 1.27)
-				)
-			)
-		)
-		(property "KiLib_Generator" "resistor/THT"
-			(at 0 0 90)
-			(layer "F.SilkS")
-			(hide yes)
-			(effects
-				(font
-					(size 1 1)
-					(thickness 0.15)
-				)
-			)
-		)
-		(property ki_fp_filters "R_*")
-		(sheetname "/")
-		(sheetfile "ZX81_Expansion_Breakout.kicad_sch")
-		(units
-			(unit
-				(name "A")
-				(pins "1" "2")
-			)
-		)
-		(attr through_hole)
-		(duplicate_pad_numbers_are_jumpers no)
-		(fp_line
-			(start 0.54 1.37)
-			(end 7.08 1.37)
-			(stroke
-				(width 0.12)
-				(type solid)
-			)
-			(layer "F.SilkS")
-		)
-		(fp_line
-			(start 7.08 1.37)
-			(end 7.08 1.04)
-			(stroke
-				(width 0.12)
-				(type solid)
-			)
-			(layer "F.SilkS")
-		)
-		(fp_line
-			(start 0.54 1.04)
-			(end 0.54 1.37)
-			(stroke
-				(width 0.12)
-				(type solid)
-			)
-			(layer "F.SilkS")
-		)
-		(fp_line
-			(start 0.54 -1.04)
-			(end 0.54 -1.37)
-			(stroke
-				(width 0.12)
-				(type solid)
-			)
-			(layer "F.SilkS")
-		)
-		(fp_line
-			(start 0.54 -1.37)
-			(end 7.08 -1.37)
-			(stroke
-				(width 0.12)
-				(type solid)
-			)
-			(layer "F.SilkS")
-		)
-		(fp_line
-			(start 7.08 -1.37)
-			(end 7.08 -1.04)
-			(stroke
-				(width 0.12)
-				(type solid)
-			)
-			(layer "F.SilkS")
-		)
-		(fp_rect
-			(start -1.05 -1.5)
-			(end 8.67 1.5)
-			(stroke
-				(width 0.05)
-				(type solid)
-			)
-			(fill no)
-			(layer "F.CrtYd")
-		)
-		(fp_line
-			(start 0 0)
-			(end 0.66 0)
-			(stroke
-				(width 0.1)
-				(type solid)
-			)
-			(layer "F.Fab")
-		)
-		(fp_line
-			(start 7.62 0)
-			(end 6.96 0)
-			(stroke
-				(width 0.1)
-				(type solid)
-			)
-			(layer "F.Fab")
-		)
-		(fp_rect
-			(start 0.66 -1.25)
-			(end 6.96 1.25)
-			(stroke
-				(width 0.1)
-				(type solid)
-			)
-			(fill no)
-			(layer "F.Fab")
-		)
-		(fp_text user "${REFERENCE}"
-			(at 3.81 0 90)
-			(layer "F.Fab")
-			(effects
-				(font
-					(size 1 1)
-					(thickness 0.15)
-				)
-			)
-		)
-		(pad "1" thru_hole circle
-			(at 0 0 270)
-			(size 1.6 1.6)
-			(drill 0.8)
-			(layers "*.Cu" "*.Mask")
-			(remove_unused_layers no)
-			(net "~{RESET}")
-			(pintype "passive")
-		)
-		(pad "2" thru_hole circle
-			(at 7.62 0 270)
-			(size 1.6 1.6)
-			(drill 0.8)
-			(layers "*.Cu" "*.Mask")
-			(remove_unused_layers no)
-			(net "Net-(R1-Pad2)")
-			(pintype "passive")
-		)
-		(embedded_fonts no)
-		(model "${KICAD10_3DMODEL_DIR}/Resistor_THT.3dshapes/R_Axial_DIN0207_L6.3mm_D2.5mm_P7.62mm_Horizontal.step"
-			(offset
-				(xyz 0 0 0)
-			)
-			(scale
-				(xyz 1 1 1)
-			)
-			(rotate
-				(xyz 0 0 0)
-			)
-		)
-	)
 	(footprint "Connector_PinHeader_2.54mm:PinHeader_2x23_P2.54mm_Vertical"
 		(layer "F.Cu")
@@
 			(remove_unused_layers no)
 			(roundrect_rratio 0.1470588235)
-			(net "Net-(R1-Pad2)")
+			(net "~{RESET}")
 			(pintype "passive")
 		)
@@
 		)
 	)
-	(gr_text "Brett Hallen, Jul 2026"
+	(gr_text "Brett Hallen, Oct 2026"
 		(at 89.662 65.024 0)
 		(layer "B.SilkS")
@@
 	)
 	(segment
-		(start 112.994 74.293)
-		(end 111.943982 75.343018)
+		(start 110.624 66.802)
+		(end 110.624 66.541)
 		(width 0.2)
 		(layer "F.Cu")
@@
 	)
 	(segment
-		(start 111.963982 44.881018)
-		(end 111.963982 33.432)
+		(start 110.624 66.802)
+		(end 111.943982 68.121982)
 		(width 0.2)
 		(layer "F.Cu")
@@
 	)
 	(segment
-		(start 112.994 55.957)
-		(end 112.994 74.293)
+		(start 111.963982 44.881018)
+		(end 111.963982 33.432)
 		(width 0.2)
 		(layer "F.Cu")
@@
 	)
 	(segment
-		(start 111.894 54.857)
-		(end 112.994 55.957)
+		(start 111.894 65.271)
+		(end 111.894 50.412)
 		(width 0.2)
 		(layer "F.Cu")
@@
 	)
 	(segment
+		(start 111.943982 68.121982)
+		(end 111.943982 78.602)
+		(width 0.2)
+		(layer "F.Cu")
+		(net "~{RESET}")
+	)
+	(segment
 		(start 111.894 50.412)
 		(end 110.744 49.262)
@@
 	)
 	(segment
-		(start 110.744 46.101)
-		(end 111.963982 44.881018)
+		(start 110.624 66.541)
+		(end 111.894 65.271)
 		(width 0.2)
 		(layer "F.Cu")
@@
 	)
 	(segment
-		(start 111.894 50.412)
-		(end 111.894 54.857)
+		(start 110.744 46.101)
+		(end 111.963982 44.881018)
 		(width 0.2)
 		(layer "F.Cu")
@@
 	)
 	(segment
-		(start 110.624 66.802)
-		(end 110.624 63.747)
-		(width 0.2)
-		(layer "F.Cu")
-		(net "Net-(R1-Pad2)")
-	)
-	(segment
-		(start 110.624 63.747)
-		(end 111.894 62.477)
-		(width 0.2)
-		(layer "F.Cu")
-		(net "Net-(R1-Pad2)")
-	)
-	(segment

Commit message: Improved PCB layout
Parts:
- removed R2: LINK, Connector_PinHeader_2.54mm:PinHeader_1x02_P2.54mm_Vertical
- moved J4 7.04 mm to (107.4, 56.1)
- moved SW1 5.86 mm to (111.9, 59.9), turned to -90 degrees
- moved J5 0.89 mm to (66.4, 56.1)
Connections:
- SW1 pad 1: Net-(SW1-A) -> ~{RESET}
Routing:
- net GND: track 100.6 -> 107.6 mm
- net Net-(SW1-A): track 4.15 -> 0.00 mm
- net ~{RESET}: track 50.5 -> 49.4 mm
Other:
- board text added: "ZX81 EXPANSION BREAKOUT ISSUE 2"
- board text added: "~{ROMCS} (A25)"
- board text removed: "ZX81 EXPANSION BREAKOUT ISSUE 1"
- board text removed: "~{ROMCS}"
