File: ZX81_Expansion_Breakout/ZX81_Expansion_Breakout.kicad_sch (KiCad schematic)
At the start: 8 parts, among them J1 ZX81 Expansion, J2 Pin Header Breakout, J3 ZX81 Extender, J4 GND LINK, J5 GND LINK, SW1 RESET

Commit message: Tested design
Removed 470Ω current limiting resistor on ~RESET line
Parts:
- removed R1: 470Ω, Resistor_THT:R_Axial_DIN0207_L6.3mm_D2.5mm_P7.62mm_Horizontal, symbol Device:R
Connections:
- net ~{RESET}: now also R2.1
Changed lines of the file:
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@@
 	(title_block
 		(title "ZX81 Expansion Breakout")
-		(date "25/JUL/2026")
-		(rev "Issue 1")
+		(date "20/Oct/2026")
+		(rev "Issue 2")
 		(company "Brett Hallen")
 		(comment 3 "https://github.com/zxinfo-diy-electronics/zx81-bus-extender")
@@
 	(wire
 		(pts
-			(xy 80.01 127) (xy 83.82 127)
+			(xy 106.68 127) (xy 101.6 127)
 		)
 		(stroke
@@
 	(wire
 		(pts
-			(xy 106.68 127) (xy 101.6 127)
+			(xy 72.39 127) (xy 83.82 127)
 		)
 		(stroke
@@
 					(unit 1)
 				)
-			)
-		)
-	)
-	(symbol
-		(lib_id "Device:R")
-		(at 76.2 127 90)
-		(unit 1)
-		(body_style 1)
-		(exclude_from_sim no)
-		(in_bom yes)
-		(on_board yes)
-		(in_pos_files yes)
-		(dnp no)
-		(fields_autoplaced yes)
-		(property "Reference" "R1"
-			(at 76.2 120.65 90)
-			(show_name no)
-			(do_not_autoplace no)
-			(effects
-				(font
-					(size 1.27 1.27)
-				)
-			)
-		)
-		(property "Value" "470Ω"
-			(at 76.2 123.19 90)
-			(show_name no)
-			(do_not_autoplace no)
-			(effects
-				(font
-					(size 1.27 1.27)
-				)
-			)
-		)
-		(property "Footprint" "Resistor_THT:R_Axial_DIN0207_L6.3mm_D2.5mm_P7.62mm_Horizontal"
-			(at 76.2 128.778 90)
-			(hide yes)
-			(show_name no)
-			(do_not_autoplace no)
-			(effects
-				(font
-					(size 1.27 1.27)
-				)
-			)
-		)
-		(property "Datasheet" ""
-			(at 76.2 127 0)
-			(hide yes)
-			(show_name no)
-			(do_not_autoplace no)
-			(effects
-				(font
-					(size 1.27 1.27)
-				)
-			)
-		)
-		(property "Description" "Resistor"
-			(at 76.2 127 0)
-			(hide yes)
-			(show_name no)
-			(do_not_autoplace no)
-			(effects
-				(font
-					(size 1.27 1.27)
-				)
-			)
-		)
-		(pin "1"
-		)
-		(pin "2"
-		)
-		(instances
-			(project "ZX81_Expansion_Breakout"
-				(path "/9fe308ca-3f7b-4728-94aa-e25b3513d2a1"
-					(reference "R1")
-					(unit 1)
-				)

Commit message: Improved PCB layout
Parts:
- removed R2: LINK, Connector_PinHeader_2.54mm:PinHeader_1x02_P2.54mm_Vertical, symbol Device:R
Connections:
- net ~{RESET}: now also SW1.1 (A)
Other:
- note added: "To get the [RESET] button to work the GND link is required, as indicated on the PCB."
- note removed: "To get the [RESET] button to work two link wires are required, as indicated on the PCB."
Changed lines of the file:
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@@
 		(comment 4 "Based on ZX81 Bus Extender by Thomas Kolbeck")
 	)
-	(text "To get the [RESET] button to work two link wires are required, as indicated on the PCB."
+	(text "To get the [RESET] button to work the GND link is required, as indicated on the PCB."
 		(exclude_from_sim no)
 		(at 94.234 138.684 0)
@@
 	(wire
 		(pts
-			(xy 72.39 127) (xy 83.82 127)
+			(xy 88.9 127) (xy 91.44 127)
 		)
 		(stroke
@@
 	(global_label "~{RESET}"
 		(shape input)
-		(at 72.39 127 180)
+		(at 88.9 127 180)
 		(fields_autoplaced yes)
 		(effects
@@
 		)
 		(property "Intersheetrefs" "${INTERSHEET_REFS}"
-			(at 63.6597 127 0)
+			(at 80.1697 127 0)
 			(hide yes)
 			(show_name no)
@@
 					(unit 1)
 				)
-			)
-		)
-	)
-	(symbol
-		(lib_id "Device:R")
-		(at 87.63 127 90)
-		(unit 1)
-		(body_style 1)
-		(exclude_from_sim no)
-		(in_bom yes)
-		(on_board yes)
-		(in_pos_files yes)
-		(dnp no)
-		(fields_autoplaced yes)
-		(property "Reference" "R2"
-			(at 87.63 120.65 90)
-			(show_name no)
-			(do_not_autoplace no)
-			(effects
-				(font
-					(size 1.27 1.27)
-				)
-			)
-		)
-		(property "Value" "LINK"
-			(at 87.63 123.19 90)
-			(show_name no)
-			(do_not_autoplace no)
-			(effects
-				(font
-					(size 1.27 1.27)
-				)
-			)
-		)
-		(property "Footprint" "Connector_PinHeader_2.54mm:PinHeader_1x02_P2.54mm_Vertical"
-			(at 87.63 128.778 90)
-			(hide yes)
-			(show_name no)
-			(do_not_autoplace no)
-			(effects
-				(font
-					(size 1.27 1.27)
-				)
-			)
-		)
-		(property "Datasheet" ""
-			(at 87.63 127 0)
-			(hide yes)
-			(show_name no)
-			(do_not_autoplace no)
-			(effects
-				(font
-					(size 1.27 1.27)
-				)
-			)
-		)
-		(property "Description" "Resistor"
-			(at 87.63 127 0)
-			(hide yes)
-			(show_name no)
-			(do_not_autoplace no)
-			(effects
-				(font
-					(size 1.27 1.27)
-				)
-			)
-		)
-		(pin "1"
-		)
-		(pin "2"
-		)
-		(instances
-			(project "ZX81_Expansion_Breakout"
-				(path "/9fe308ca-3f7b-4728-94aa-e25b3513d2a1"
-					(reference "R2")
-					(unit 1)
-				)
